File: power.sch (KiCad schematic (older format))
At the start: 13 parts

Commit message: Passing ERC
Parts:
- removed C? (x2): 2.2u, w_smd_cap:c_0805, symbol C
- removed U?: LP38691, knielsenlib:TO-252-3, symbol LP38691
- added C19: 22n, symbol C_Small
- added C23: 1u, symbol C_Small
- added C24: 2u2, symbol C_Small
- added C25: 10n, symbol C_Small
- added U5: LP2985LV, symbol LP2985LV
- R31: renamed from R?; value R_Small -> 15k
- R32: renamed from R?; value R_Small -> 3k3
- R33: renamed from R?; value R_Small -> 4k7
- gave numbers to parts that had none: 7
Connections:
- net +3V3: now also C24.1, U5.5 (VOUT)
- net GND: now also C23.2, C24.2, C25.2, U5.2 (GND)
- net VCC: now also C23.1, U5.1 (VIN), U5.3 (ON/OFF)
- net at L2.1, U6.1 (VSW), U6.12 (VSW)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: now also C19.2; no longer U6.10 (BST)
- new net: C19.1, U6.10 (BST)
- new net bypass: C25.1, U5.4 (BYPASS)
Other:
- note added: "Buck converter"
- note added: "Jumper 1-2 powers logic from motor supply\nJumper 3-4 powers logic from buck converter\nJumper 5-6 powers logic from USB"
- note removed: "Jumper 1-2 powers logic from motor supply\nJumper 3-4 power logic from buck converter\nJumper 5-6 powers logic from USB"
- moved on the sheet: C20, C21, C22, L2, P5, P6, R31, R32, R33, U6

Commit message: Starting on netlist
Parts:
- C19: footprint (none) -> Capacitors_SMD:C_0603
- C20, C21, C22, C23, C24, C25: footprint (none) -> Capacitors_SMD:C_0805
- L2: footprint (none) -> Inductors_SMD:L_7.3x7.3_H3.5
- P5: footprint (none) -> Pin_Headers:Pin_Header_Straight_2x03_Pitch1.27mm
- P6: footprint (none) -> knielsenlib:con-jack-DCJ0303
- R31, R32, R33: footprint (none) -> Resistors_SMD:R_0603
- U5: footprint (none) -> TO_SOT_Packages_SMD:SOT-23-5
- U6: footprint (none) -> Housings_DFN_QFN:QFN-16-1EP_3x3mm_Pitch0.5mm
Changed lines of the file:
@@
 LIBS:w_device
 LIBS:pcb_ledtorus_controller-cache
-LIBS:tiva_pcb1-cache
 EELAYER 26 0
 EELAYER END
@@
 F 0 "U6" H 2200 3043 60  0000 C CNN
 F 1 "TS3001x" H 2200 2910 90  0000 C CNN
-F 2 "" H 2300 2300 60  0001 C CNN
+F 2 "Housings_DFN_QFN:QFN-16-1EP_3x3mm_Pitch0.5mm" H 2300 2300 60  0001 C CNN
 F 3 "" H 2300 2300 60  0001 C CNN
 	1    2200 2200
@@
 F 0 "C20" H 1492 2047 50  0000 L CNN
 F 1 "10u" H 1492 1954 50  0000 L CNN
-F 2 "" H 1400 2000 50  0001 C CNN
+F 2 "Capacitors_SMD:C_0805" H 1400 2000 50  0001 C CNN
 F 3 "" H 1400 2000 50  0001 C CNN
 	1    1400 2000
@@
 F 0 "C21" H 3392 2047 50  0000 L CNN
 F 1 "22u" H 3392 1954 50  0000 L CNN
-F 2 "" H 3300 2000 50  0001 C CNN
+F 2 "Capacitors_SMD:C_0805" H 3300 2000 50  0001 C CNN
 F 3 "" H 3300 2000 50  0001 C CNN
 	1    3300 2000
@@
 F 0 "R31" H 3059 2347 50  0000 L CNN
 F 1 "15k" H 3059 2254 50  0000 L CNN
-F 2 "" H 3000 2300 50  0001 C CNN
+F 2 "Resistors_SMD:R_0603" H 3000 2300 50  0001 C CNN
 F 3 "" H 3000 2300 50  0001 C CNN
 	1    3000 2300
@@
 F 0 "R32" H 2850 2750 50  0000 L CNN
 F 1 "3k3" H 2800 2650 50  0000 L CNN
-F 2 "" H 3000 2700 50  0001 C CNN
+F 2 "Resistors_SMD:R_0603" H 3000 2700 50  0001 C CNN
 F 3 "" H 3000 2700 50  0001 C CNN
 	1    3000 2700
@@
 F 0 "C22" H 3692 2047 50  0000 L CNN
 F 1 "22u" H 3692 1954 50  0000 L CNN
-F 2 "" H 3600 2000 50  0001 C CNN
+F 2 "Capacitors_SMD:C_0805" H 3600 2000 50  0001 C CNN
 F 3 "" H 3600 2000 50  0001 C CNN
 	1    3600 2000
@@
 F 0 "L2" V 3291 1900 50  0000 C CNN
 F 1 "4u7" V 3198 1900 50  0000 C CNN
-F 2 "" H 3100 1900 50  0001 C CNN
+F 2 "Inductors_SMD:L_7.3x7.3_H3.5" H 3100 1900 50  0001 C CNN
 F 3 "" H 3100 1900 50  0001 C CNN
 	1    3100 1900
@@
 F 0 "R33" H 3259 2747 50  0000 L CNN
 F 1 "4k7" H 3259 2654 50  0000 L CNN
-F 2 "" H 3200 2700 50  0001 C CNN
+F 2 "Resistors_SMD:R_0603" H 3200 2700 50  0001 C CNN
 F 3 "" H 3200 2700 50  0001 C CNN
 	1    3200 2700
@@
 F 0 "P5" H 2650 4800 50  0000 C CNN
 F 1 "CONN_3X2" V 2650 4600 40  0000 C CNN
-F 2 "" H 2650 4550 60  0000 C CNN
+F 2 "Pin_Headers:Pin_Header_Straight_2x03_Pitch1.27mm" H 2650 4550 60  0001 C CNN
 F 3 "" H 2650 4550 60  0000 C CNN
 	1    2650 4550
@@
 F 0 "P6" V 5100 4600 50  0000 C CNN
 F 1 "CONN_3" V 5200 4600 40  0000 C CNN
-F 2 "" H 5150 4600 60  0001 C CNN
+F 2 "knielsenlib:con-jack-DCJ0303" H 5150 4600 60  0001 C CNN
 F 3 "" H 5150 4600 60  0001 C CNN
 	1    5150 4600
@@
 F 0 "U5" H 6700 2646 60  0000 C CNN
 F 1 "LP2985LV" H 6700 2536 60  0000 C CNN
-F 2 "" H 6700 2050 60  0000 C CNN
+F 2 "TO_SOT_Packages_SMD:SOT-23-5" H 6700 2050 60  0001 C CNN
 F 3 "" H 6700 2050 60  0000 C CNN
 	1    6700 2050
@@
 F 0 "C25" H 5792 2497 50  0000 L CNN
 F 1 "10n" H 5792 2404 50  0000 L CNN
-F 2 "" H 5700 2450 50  0001 C CNN
+F 2 "Capacitors_SMD:C_0805" H 5700 2450 50  0001 C CNN
 F 3 "" H 5700 2450 50  0001 C CNN
 	1    5700 2450
@@
 F 0 "C23" H 5692 2097 50  0000 L CNN
 F 1 "1u" H 5692 2004 50  0000 L CNN
-F 2 "" H 5600 2050 50  0001 C CNN
+F 2 "Capacitors_SMD:C_0805" H 5600 2050 50  0001 C CNN
 F 3 "" H 5600 2050 50  0001 C CNN
 	1    5600 2050
@@
 F 0 "C24" H 7692 2097 50  0000 L CNN
 F 1 "2u2" H 7692 2004 50  0000 L CNN
-F 2 "" H 7600 2050 50  0001 C CNN
+F 2 "Capacitors_SMD:C_0805" H 7600 2050 50  0001 C CNN
 F 3 "" H 7600 2050 50  0001 C CNN
 	1    7600 2050
@@
 F 0 "C19" H 2750 1850 50  0000 L CNN
 F 1 "22n" H 2700 1750 50  0000 L CNN
-F 2 "" H 2900 1800 50  0001 C CNN
+F 2 "Capacitors_SMD:C_0603" H 2900 1800 50  0001 C CNN
 F 3 "" H 2900 1800 50  0001 C CNN
 	1    2900 1800

Commit message: Starting on netlist
Parts:
- P5: footprint Pin_Headers:Pin_Header_Straight_2x03_Pitch1.27mm -> Pin_Headers:Pin_Header_Straight_2x03_Pitch2.54mm
Changed lines of the file:
@@
 LIBS:contrib
 LIBS:valves
-LIBS:w_analog
-LIBS:w_device
 LIBS:pcb_ledtorus_controller-cache
 EELAYER 26 0
@@
 F 0 "P5" H 2650 4800 50  0000 C CNN
 F 1 "CONN_3X2" V 2650 4600 40  0000 C CNN
-F 2 "Pin_Headers:Pin_Header_Straight_2x03_Pitch1.27mm" H 2650 4550 60  0001 C CNN
+F 2 "Pin_Headers:Pin_Header_Straight_2x03_Pitch2.54mm" H 2650 4550 60  0001 C CNN
 F 3 "" H 2650 4550 60  0000 C CNN
 	1    2650 4550

Commit message: Work on layout
Parts:
- P6: footprint knielsenlib:con-jack-DCJ0303 -> w_conn_misc:dc_socket
Connections:
- net +24V: now also P5.3; no longer P5.1
- net +8V: now also P5.5; no longer P5.3
- net usb5v: now also P5.1; no longer P5.5
- net vsw: now reaches C19.2, L2.1, U6.1 (VSW), U6.12 (VSW), U6.13 (VSW), U6.16 (VSW)
- net fb: now reaches R31.2, R32.1, R33.1, U6.5 (FB)
Changed lines of the file:
@@
 L +24V #PWR048
 U 1 1 5C27B179
-P 1950 4300
-F 0 "#PWR048" H 1950 4150 50  0001 C CNN
-F 1 "+24V" H 1965 4477 50  0000 C CNN
-F 2 "" H 1950 4300 50  0001 C CNN
-F 3 "" H 1950 4300 50  0001 C CNN
-	1    1950 4300
-	1    0    0    -1
-$EndComp
-Text GLabel 1950 4600 0    60   Input ~ 0
+P 1750 4400
+F 0 "#PWR048" H 1750 4250 50  0001 C CNN
+F 1 "+24V" H 1765 4577 50  0000 C CNN
+F 2 "" H 1750 4400 50  0001 C CNN
+F 3 "" H 1750 4400 50  0001 C CNN
+	1    1750 4400
+	1    0    0    -1
+$EndComp
+Text GLabel 2150 4400 0    60   Input ~ 0
 usb5v
 $Comp
@@
 F 0 "P6" V 5100 4600 50  0000 C CNN
 F 1 "CONN_3" V 5200 4600 40  0000 C CNN
-F 2 "knielsenlib:con-jack-DCJ0303" H 5150 4600 60  0001 C CNN
+F 2 "w_conn_misc:dc_socket" H 5150 4600 60  0001 C CNN
 F 3 "" H 5150 4600 60  0001 C CNN
 	1    5150 4600
@@
 L +8V #PWR047
 U 1 1 5C27DC56
-P 1750 4300
-F 0 "#PWR047" H 1750 4150 50  0001 C CNN
-F 1 "+8V" H 1765 4477 50  0000 C CNN
-F 2 "" H 1750 4300 50  0001 C CNN
-F 3 "" H 1750 4300 50  0001 C CNN
-	1    1750 4300
+P 1550 4400
+F 0 "#PWR047" H 1550 4250 50  0001 C CNN
+F 1 "+8V" H 1565 4577 50  0000 C CNN
+F 2 "" H 1550 4400 50  0001 C CNN
+F 3 "" H 1550 4400 50  0001 C CNN
+	1    1550 4400
 	1    0    0    -1
 $EndComp
@@
 	3050 4400 3400 4400
 Wire Wire Line
-	1950 4600 2250 4600
-Wire Wire Line
-	2250 4400 1950 4400
-Wire Wire Line
-	1950 4400 1950 4300
+	2150 4400 2250 4400
+Wire Wire Line
+	1750 4500 2250 4500
+Wire Wire Line
+	1750 4500 1750 4400
 Connection ~ 4650 4500
 Wire Wire Line
@@
 	4450 4500 4450 4400
 Wire Wire Line
-	2250 4500 1750 4500
-Wire Wire Line
-	1750 4500 1750 4300
+	1550 4600 2250 4600
+Wire Wire Line
+	1550 4600 1550 4400
 Wire Wire Line
 	5700 2350 5700 2250
@@
 	5700 2250 5900 2250
 Wire Wire Line
-	5700 2550 5700 2750
+	5700 2750 5700 2550
 Wire Wire Line
 	5500 2750 7600 2750
@@
 	1    0    0    -1
 $EndComp
+Text Label 2950 1900 0    30   ~ 0
+vsw
+Text Label 3050 2500 0    30   ~ 0
+fb
 $EndSCHEMATC

Commit message: Completing cleanups and ToDos:
 - L6234 thermal vias done
 - Gerbers checked
 - Misc. io and stuff tweaks
Parts:
- L2: footprint Inductors_SMD:L_7.3x7.3_H3.5 -> knielsenlib:Coil_WE_7447786004
- P6: footprint w_conn_misc:dc_socket -> knielsenlib:dc_socket
- U6: footprint Housings_DFN_QFN:QFN-16-1EP_3x3mm_Pitch0.5mm -> knielsenlib:QFN16-TS30001
Changed lines of the file:
@@
 F 0 "U6" H 2200 3043 60  0000 C CNN
 F 1 "TS3001x" H 2200 2910 90  0000 C CNN
-F 2 "Housings_DFN_QFN:QFN-16-1EP_3x3mm_Pitch0.5mm" H 2300 2300 60  0001 C CNN
+F 2 "knielsenlib:QFN16-TS30001" H 2300 2300 60  0001 C CNN
 F 3 "" H 2300 2300 60  0001 C CNN
 	1    2200 2200
@@
 F 0 "L2" V 3291 1900 50  0000 C CNN
 F 1 "4u7" V 3198 1900 50  0000 C CNN
-F 2 "Inductors_SMD:L_7.3x7.3_H3.5" H 3100 1900 50  0001 C CNN
+F 2 "knielsenlib:Coil_WE_7447786004" H 3100 1900 50  0001 C CNN
 F 3 "" H 3100 1900 50  0001 C CNN
 	1    3100 1900
@@
 F 0 "P6" V 5100 4600 50  0000 C CNN
 F 1 "CONN_3" V 5200 4600 40  0000 C CNN
-F 2 "w_conn_misc:dc_socket" H 5150 4600 60  0001 C CNN
+F 2 "knielsenlib:dc_socket" H 5150 4600 60  0001 C CNN
 F 3 "" H 5150 4600 60  0001 C CNN
 	1    5150 4600
