File: motor.sch (KiCad schematic (older format))
At the start: 31 parts

Commit message: Passing ERC
Parts:
- gave numbers to parts that had none: 31
Other:
- moved on the sheet: R23, R24

Commit message: Starting on netlist
Parts:
- C14, C15: footprint (none) -> Capacitors_SMD:C_0603
- C16, C17, C18: footprint (none) -> Capacitors_SMD:C_0805
- D3, D5, D6, D7: footprint Discret:D4 -> Diodes_SMD:D_SOD-123F
- D4: footprint (none) -> TO_SOT_Packages_SMD:SOT-23
- J1: footprint (none) -> Pin_Headers:Pin_Header_Straight_1x04_Pitch1.27mm
- R10, R11, R15, R16, R23, R24, R9: footprint (none) -> Resistors_SMD:R_0805
- R12, R13, R14: footprint Resistors_ThroughHole:Resistor_Horizontal_RM10mm -> Resistors_SMD:R_0612
- R17, R18, R19, R20, R21, R22, R6, R7, R8: footprint Resistors_ThroughHole:Resistor_Horizontal_RM10mm -> Resistors_SMD:R_0603
- U4: footprint (none) -> knielsenlib:POWERSO20
Changed lines of the file:
@@
 LIBS:w_device
 LIBS:pcb_ledtorus_controller-cache
-LIBS:tiva_pcb1-cache
 EELAYER 26 0
 EELAYER END
@@
 F 0 "U4" H 3000 2750 60  0000 C CNN
 F 1 "L6234" H 3100 4000 60  0000 C CNN
-F 2 "" H 3100 3300 60  0000 C CNN
+F 2 "knielsenlib:POWERSO20" H 3100 3300 60  0001 C CNN
 F 3 "" H 3100 3300 60  0000 C CNN
 	1    3100 3350
@@
 F 0 "C18" H 2325 4000 30  0000 L CNN
 F 1 "1u" H 2325 3900 30  0000 L CNN
-F 2 "" H 2300 3950 60  0000 C CNN
+F 2 "Capacitors_SMD:C_0805" H 2300 3950 60  0001 C CNN
 F 3 "" H 2300 3950 60  0000 C CNN
 	1    2300 3950
@@
 F 0 "C17" H 3975 2850 30  0000 L CNN
 F 1 "10n" H 3975 2750 30  0000 L CNN
-F 2 "" H 3950 2800 60  0000 C CNN
+F 2 "Capacitors_SMD:C_0805" H 3950 2800 60  0001 C CNN
 F 3 "" H 3950 2800 60  0000 C CNN
 	1    3950 2800
@@
 F 0 "C16" H 4775 2750 30  0000 L CNN
 F 1 "220n" H 4775 2650 30  0000 L CNN
-F 2 "" H 4750 2700 60  0000 C CNN
+F 2 "Capacitors_SMD:C_0805" H 4750 2700 60  0001 C CNN
 F 3 "" H 4750 2700 60  0000 C CNN
 	1    4750 2700
@@
 F 0 "C14" H 3375 2450 30  0000 L CNN
 F 1 "100n" H 3375 2350 30  0000 L CNN
-F 2 "" H 3350 2400 60  0000 C CNN
+F 2 "Capacitors_SMD:C_0603" H 3350 2400 60  0001 C CNN
 F 3 "" H 3350 2400 60  0000 C CNN
 	1    3350 2400
@@
 F 0 "R15" V 4630 3050 40  0000 C CNN
 F 1 "0R22" V 4557 3051 40  0000 C CNN
-F 2 "" V 4480 3050 30  0000 C CNN
+F 2 "Resistors_SMD:R_0805" V 4480 3050 30  0001 C CNN
 F 3 "" H 4550 3050 30  0000 C CNN
 	1    4550 3050
@@
 F 0 "R16" V 4450 3150 40  0000 C CNN
 F 1 "0R22" V 4557 3151 40  0000 C CNN
-F 2 "" V 4480 3150 30  0000 C CNN
+F 2 "Resistors_SMD:R_0805" V 4480 3150 30  0001 C CNN
 F 3 "" H 4550 3150 30  0000 C CNN
 	1    4550 3150
@@
 F 0 "R11" V 1980 2450 40  0000 C CNN
 F 1 "47k" V 1907 2451 40  0000 C CNN
-F 2 "" V 1830 2450 30  0000 C CNN
+F 2 "Resistors_SMD:R_0805" V 1830 2450 30  0001 C CNN
 F 3 "" H 1900 2450 30  0000 C CNN
 	1    1900 2450
@@
 F 0 "R10" V 1830 2450 40  0000 C CNN
 F 1 "47k" V 1757 2451 40  0000 C CNN
-F 2 "" V 1680 2450 30  0000 C CNN
+F 2 "Resistors_SMD:R_0805" V 1680 2450 30  0001 C CNN
 F 3 "" H 1750 2450 30  0000 C CNN
 	1    1750 2450
@@
 F 0 "R9" V 1680 2450 40  0000 C CNN
 F 1 "47k" V 1607 2451 40  0000 C CNN
-F 2 "" V 1530 2450 30  0000 C CNN
+F 2 "Resistors_SMD:R_0805" V 1530 2450 30  0001 C CNN
 F 3 "" H 1600 2450 30  0000 C CNN
 	1    1600 2450
@@
 F 0 "D4" H 4150 2350 40  0000 C CNN
 F 1 "BAV99LT3G" H 4050 2550 40  0000 C CNN
-F 2 "" H 4050 2450 60  0000 C CNN
+F 2 "TO_SOT_Packages_SMD:SOT-23" H 4050 2450 60  0001 C CNN
 F 3 "" H 4050 2450 60  0000 C CNN
 	1    4050 2450
@@
 F 0 "C15" H 3000 2550 30  0000 L CNN
 F 1 "100u" H 3000 2400 30  0000 L CNN
-F 2 "" H 3150 2450 60  0000 C CNN
+F 2 "Capacitors_SMD:C_0603" H 3150 2450 60  0001 C CNN
 F 3 "" H 3150 2450 60  0000 C CNN
 	1    3150 2450
@@
 F 0 "R23" V 3630 4700 40  0000 C CNN
 F 1 "0" V 3557 4701 40  0000 C CNN
-F 2 "" V 3480 4700 30  0000 C CNN
+F 2 "Resistors_SMD:R_0805" V 3480 4700 30  0001 C CNN
 F 3 "" H 3550 4700 30  0000 C CNN
 	1    3550 4700
@@
 F 0 "R24" V 3630 4900 40  0000 C CNN
 F 1 "0" V 3557 4901 40  0000 C CNN
-F 2 "" V 3480 4900 30  0000 C CNN
+F 2 "Resistors_SMD:R_0805" V 3480 4900 30  0001 C CNN
 F 3 "" H 3550 4900 30  0000 C CNN
 	1    3550 4900
@@
 F 0 "J1" V 1571 4331 50  0000 L CNN
 F 1 "CONN_01X04" V 1850 3900 50  0000 L CNN
-F 2 "" H 1700 4100 50  0001 C CNN
+F 2 "Pin_Headers:Pin_Header_Straight_1x04_Pitch1.27mm" H 1700 4100 50  0001 C CNN
 F 3 "" H 1700 4100 50  0001 C CNN
 	1    1700 4100
@@
 F 0 "R6" V 6650 2050 50  0000 C CNN
 F 1 "5k" V 6750 2050 50  0000 C CNN
-F 2 "Resistors_ThroughHole:Resistor_Horizontal_RM10mm" V 6680 2050 50  0001 C CNN
+F 2 "Resistors_SMD:R_0603" V 6680 2050 50  0001 C CNN
 F 3 "" H 6750 2050 50  0000 C CNN
 	1    6750 2050
@@
 F 0 "R7" V 7350 2050 50  0000 C CNN
 F 1 "5k" V 7450 2050 50  0000 C CNN
-F 2 "Resistors_ThroughHole:Resistor_Horizontal_RM10mm" V 7380 2050 50  0001 C CNN
+F 2 "Resistors_SMD:R_0603" V 7380 2050 50  0001 C CNN
 F 3 "" H 7450 2050 50  0000 C CNN
 	1    7450 2050
@@
 F 0 "R8" V 8050 2050 50  0000 C CNN
 F 1 "2k2" V 8150 2050 50  0000 C CNN
-F 2 "Resistors_ThroughHole:Resistor_Horizontal_RM10mm" V 8080 2050 50  0001 C CNN
+F 2 "Resistors_SMD:R_0603" V 8080 2050 50  0001 C CNN
 F 3 "" H 8150 2050 50  0000 C CNN
 	1    8150 2050
@@
 F 0 "R12" V 6650 2650 50  0000 C CNN
 F 1 "5k" V 6750 2650 50  0000 C CNN
-F 2 "Resistors_ThroughHole:Resistor_Horizontal_RM10mm" V 6680 2650 50  0001 C CNN
+F 2 "Resistors_SMD:R_0612" V 6680 2650 50  0001 C CNN
 F 3 "" H 6750 2650 50  0000 C CNN
 	1    6750 2650
@@
 F 0 "R13" V 7350 2650 50  0000 C CNN
 F 1 "5k" V 7450 2650 50  0000 C CNN
-F 2 "Resistors_ThroughHole:Resistor_Horizontal_RM10mm" V 7380 2650 50  0001 C CNN
+F 2 "Resistors_SMD:R_0612" V 7380 2650 50  0001 C CNN
 F 3 "" H 7450 2650 50  0000 C CNN
 	1    7450 2650
@@
 F 0 "R14" V 8050 2650 50  0000 C CNN
 F 1 "2k2" V 8150 2650 50  0000 C CNN
-F 2 "Resistors_ThroughHole:Resistor_Horizontal_RM10mm" V 8080 2650 50  0001 C CNN
+F 2 "Resistors_SMD:R_0612" V 8080 2650 50  0001 C CNN
 F 3 "" H 8150 2650 50  0000 C CNN
 	1    8150 2650
@@
 F 0 "R17" V 6650 3250 50  0000 C CNN
 F 1 "5k" V 6750 3250 50  0000 C CNN
-F 2 "Resistors_ThroughHole:Resistor_Horizontal_RM10mm" V 6680 3250 50  0001 C CNN
+F 2 "Resistors_SMD:R_0603" V 6680 3250 50  0001 C CNN
 F 3 "" H 6750 3250 50  0000 C CNN
 	1    6750 3250
@@
 F 0 "R18" V 7350 3250 50  0000 C CNN
 F 1 "5k" V 7450 3250 50  0000 C CNN
-F 2 "Resistors_ThroughHole:Resistor_Horizontal_RM10mm" V 7380 3250 50  0001 C CNN
+F 2 "Resistors_SMD:R_0603" V 7380 3250 50  0001 C CNN
 F 3 "" H 7450 3250 50  0000 C CNN
 	1    7450 3250
@@
 F 0 "R19" V 8050 3250 50  0000 C CNN
 F 1 "2k2" V 8150 3250 50  0000 C CNN
-F 2 "Resistors_ThroughHole:Resistor_Horizontal_RM10mm" V 8080 3250 50  0001 C CNN
+F 2 "Resistors_SMD:R_0603" V 8080 3250 50  0001 C CNN
 F 3 "" H 8150 3250 50  0000 C CNN
 	1    8150 3250
@@
 F 0 "R20" V 6650 3850 50  0000 C CNN
 F 1 "5k" V 6750 3850 50  0000 C CNN
-F 2 "Resistors_ThroughHole:Resistor_Horizontal_RM10mm" V 6680 3850 50  0001 C CNN
+F 2 "Resistors_SMD:R_0603" V 6680 3850 50  0001 C CNN
 F 3 "" H 6750 3850 50  0000 C CNN
 	1    6750 3850
@@
 F 0 "R21" V 7350 3850 50  0000 C CNN
 F 1 "5k" V 7450 3850 50  0000 C CNN
-F 2 "Resistors_ThroughHole:Resistor_Horizontal_RM10mm" V 7380 3850 50  0001 C CNN
+F 2 "Resistors_SMD:R_0603" V 7380 3850 50  0001 C CNN
 F 3 "" H 7450 3850 50  0000 C CNN
 	1    7450 3850
@@
 F 0 "R22" V 8050 3850 50  0000 C CNN
 F 1 "2k2" V 8150 3850 50  0000 C CNN
-F 2 "Resistors_ThroughHole:Resistor_Horizontal_RM10mm" V 8080 3850 50  0001 C CNN
+F 2 "Resistors_SMD:R_0603" V 8080 3850 50  0001 C CNN
 F 3 "" H 8150 3850 50  0000 C CNN
 	1    8150 3850
@@
 F 0 "D3" V 7103 2321 50  0000 L CNN
 F 1 "7V" V 7196 2321 50  0000 L CNN
-F 2 "Discret:D4" H 7150 2250 50  0001 C CNN
+F 2 "Diodes_SMD:D_SOD-123F" H 7150 2250 50  0001 C CNN
 F 3 "" H 7150 2250 50  0000 C CNN
 	1    7150 2250
@@
 F 0 "D5" V 7103 2921 50  0000 L CNN
 F 1 "7V" V 7196 2921 50  0000 L CNN
-F 2 "Discret:D4" H 7150 2850 50  0001 C CNN
+F 2 "Diodes_SMD:D_SOD-123F" H 7150 2850 50  0001 C CNN
 F 3 "" H 7150 2850 50  0000 C CNN
 	1    7150 2850
@@
 F 0 "D6" V 7103 3521 50  0000 L CNN
 F 1 "7V" V 7196 3521 50  0000 L CNN
-F 2 "Discret:D4" H 7150 3450 50  0001 C CNN
+F 2 "Diodes_SMD:D_SOD-123F" H 7150 3450 50  0001 C CNN
 F 3 "" H 7150 3450 50  0000 C CNN
 	1    7150 3450
@@
 F 0 "D7" V 7103 4121 50  0000 L CNN
 F 1 "7V" V 7196 4121 50  0000 L CNN
-F 2 "Discret:D4" H 7150 4050 50  0001 C CNN
+F 2 "Diodes_SMD:D_SOD-123F" H 7150 4050 50  0001 C CNN
 F 3 "" H 7150 4050 50  0000 C CNN
 	1    7150 4050

Commit message: Starting on netlist
Parts:
- J1: footprint Pin_Headers:Pin_Header_Straight_1x04_Pitch1.27mm -> Pin_Headers:Pin_Header_Straight_1x04_Pitch2.54mm
Changed lines of the file:
@@
 LIBS:contrib
 LIBS:valves
-LIBS:w_analog
-LIBS:w_device
 LIBS:pcb_ledtorus_controller-cache
 EELAYER 26 0
@@
 F 0 "J1" V 1571 4331 50  0000 L CNN
 F 1 "CONN_01X04" V 1850 3900 50  0000 L CNN
-F 2 "Pin_Headers:Pin_Header_Straight_1x04_Pitch1.27mm" H 1700 4100 50  0001 C CNN
+F 2 "Pin_Headers:Pin_Header_Straight_1x04_Pitch2.54mm" H 1700 4100 50  0001 C CNN
 F 3 "" H 1700 4100 50  0001 C CNN
 	1    1700 4100

Commit message: Work on layout
Parts:
- C15: footprint Capacitors_SMD:C_0603 -> w_smd_cap:c_elec_6.3x5.3
- D3, D5, D6, D7: footprint Diodes_SMD:D_SOD-123F -> Diodes_SMD:D_SOD-123
- R12, R13, R14: footprint Resistors_SMD:R_0612 -> Resistors_SMD:R_0603
Changed lines of the file:
@@
 F 0 "C15" H 3000 2550 30  0000 L CNN
 F 1 "100u" H 3000 2400 30  0000 L CNN
-F 2 "Capacitors_SMD:C_0603" H 3150 2450 60  0001 C CNN
+F 2 "w_smd_cap:c_elec_6.3x5.3" H 3150 2450 60  0001 C CNN
 F 3 "" H 3150 2450 60  0000 C CNN
 	1    3150 2450
@@
 F 0 "R12" V 6650 2650 50  0000 C CNN
 F 1 "5k" V 6750 2650 50  0000 C CNN
-F 2 "Resistors_SMD:R_0612" V 6680 2650 50  0001 C CNN
+F 2 "Resistors_SMD:R_0603" V 6680 2650 50  0001 C CNN
 F 3 "" H 6750 2650 50  0000 C CNN
 	1    6750 2650
@@
 F 0 "R13" V 7350 2650 50  0000 C CNN
 F 1 "5k" V 7450 2650 50  0000 C CNN
-F 2 "Resistors_SMD:R_0612" V 7380 2650 50  0001 C CNN
+F 2 "Resistors_SMD:R_0603" V 7380 2650 50  0001 C CNN
 F 3 "" H 7450 2650 50  0000 C CNN
 	1    7450 2650
@@
 F 0 "R14" V 8050 2650 50  0000 C CNN
 F 1 "2k2" V 8150 2650 50  0000 C CNN
-F 2 "Resistors_SMD:R_0612" V 8080 2650 50  0001 C CNN
+F 2 "Resistors_SMD:R_0603" V 8080 2650 50  0001 C CNN
 F 3 "" H 8150 2650 50  0000 C CNN
 	1    8150 2650
@@
 F 0 "D3" V 7103 2321 50  0000 L CNN
 F 1 "7V" V 7196 2321 50  0000 L CNN
-F 2 "Diodes_SMD:D_SOD-123F" H 7150 2250 50  0001 C CNN
+F 2 "Diodes_SMD:D_SOD-123" H 7150 2250 50  0001 C CNN
 F 3 "" H 7150 2250 50  0000 C CNN
 	1    7150 2250
@@
 F 0 "D5" V 7103 2921 50  0000 L CNN
 F 1 "7V" V 7196 2921 50  0000 L CNN
-F 2 "Diodes_SMD:D_SOD-123F" H 7150 2850 50  0001 C CNN
+F 2 "Diodes_SMD:D_SOD-123" H 7150 2850 50  0001 C CNN
 F 3 "" H 7150 2850 50  0000 C CNN
 	1    7150 2850
@@
 F 0 "D6" V 7103 3521 50  0000 L CNN
 F 1 "7V" V 7196 3521 50  0000 L CNN
-F 2 "Diodes_SMD:D_SOD-123F" H 7150 3450 50  0001 C CNN
+F 2 "Diodes_SMD:D_SOD-123" H 7150 3450 50  0001 C CNN
 F 3 "" H 7150 3450 50  0000 C CNN
 	1    7150 3450
@@
 F 0 "D7" V 7103 4121 50  0000 L CNN
 F 1 "7V" V 7196 4121 50  0000 L CNN
-F 2 "Diodes_SMD:D_SOD-123F" H 7150 4050 50  0001 C CNN
+F 2 "Diodes_SMD:D_SOD-123" H 7150 4050 50  0001 C CNN
 F 3 "" H 7150 4050 50  0000 C CNN
 	1    7150 4050

Commit message: Submitted rev1 for production @ SeeedStudio
Parts:
- C15: footprint w_smd_cap:c_elec_6.3x5.3 -> w_smd_cap:c_elec_6.3x7.7
- U4: footprint knielsenlib:POWERSO20 -> knielsenlib:POWERSO20_stencil
Changed lines of the file:
@@
 F 0 "U4" H 3000 2750 60  0000 C CNN
 F 1 "L6234" H 3100 4000 60  0000 C CNN
-F 2 "knielsenlib:POWERSO20" H 3100 3300 60  0001 C CNN
+F 2 "knielsenlib:POWERSO20_stencil" H 3100 3300 60  0001 C CNN
 F 3 "" H 3100 3300 60  0000 C CNN
 	1    3100 3350
@@
 F 0 "C15" H 3000 2550 30  0000 L CNN
 F 1 "100u" H 3000 2400 30  0000 L CNN
-F 2 "w_smd_cap:c_elec_6.3x5.3" H 3150 2450 60  0001 C CNN
+F 2 "w_smd_cap:c_elec_6.3x7.7" H 3150 2450 60  0001 C CNN
 F 3 "" H 3150 2450 60  0000 C CNN
 	1    3150 2450
